File: pcb/DHFrontPanel/DH_LEDRing/DH_LEDRing.sch (KiCad schematic (older format))
At the start: 4 parts

Commit message: Pushing layout work
Parts:
- added C1: 0.1uF, Capacitor_SMD:C_0603_1608Metric, symbol Device:C
- added C2: 10uF, Capacitor_SMD:C_0603_1608Metric, symbol Device:C
- added D10, D11, D12, D13, D14, D15, D5, D6, D7, D8, D9: APA102-2020, LED_SMD:LED-APA102-2020, symbol LED:APA102-2020
- added J1: Conn_01x07_Male, Connector_PinHeader_2.54mm:PinHeader_1x07_P2.54mm_Vertical, symbol Connector:Conn_01x07_Male
- added J2: Conn_01x03_Male, Connector_PinHeader_2.54mm:PinHeader_1x03_P2.54mm_Vertical, symbol Connector:Conn_01x03_Male
- added RV1: 10k, Potentiometer_THT:Potentiometer_Alps_RK09L_Single_Vertical, symbol Device:R_POT
Connections:
- net GND: now also J2.3 (Pin_3), RV1.3; no longer D1.6 (GND), D2.6 (GND), D3.6 (GND), D4.6 (GND)
- net VDD: now also C1.1, C2.1, D10.1 (VDD), D11.1 (VDD), D12.1 (VDD), D13.1 (VDD), D14.1 (VDD), D15.1 (VDD), D5.1 (VDD), D6.1 (VDD), D7.1 (VDD), D8.1 (VDD), D9.1 (VDD), J1.4 (Pin_4)
- net SDI: now reaches D1.4 (SDI)
- net SDI: now also J1.2 (Pin_2)
- net CKI: now reaches D1.5 (CKI)
- net CKI: now also J1.3 (Pin_3)
- net at D4.2 (CKO): now also D5.5 (CKI)
- net at D4.3 (SDO): now also D5.4 (SDI)
- new net: D5.2 (CKO), D6.5 (CKI)
- new net: D5.3 (SDO), D6.4 (SDI)
- new net: D6.2 (CKO), D7.5 (CKI)
- new net: D6.3 (SDO), D7.4 (SDI)
- new net: D7.2 (CKO), D8.5 (CKI)
- new net: D7.3 (SDO), D8.4 (SDI)
- new net: D8.2 (CKO), D9.5 (CKI)
- new net: D8.3 (SDO), D9.4 (SDI)
- new net: D10.5 (CKI), D9.2 (CKO)
- new net: D10.4 (SDI), D9.3 (SDO)
- new net: D10.2 (CKO), D11.5 (CKI)
- new net: D10.3 (SDO), D11.4 (SDI)
- new net: D11.2 (CKO), D12.5 (CKI)
- new net: D11.3 (SDO), D12.4 (SDI)
- new net: D12.2 (CKO), D13.5 (CKI)
- new net: D12.3 (SDO), D13.4 (SDI)
- new net: D13.2 (CKO), D14.5 (CKI)
- new net: D13.3 (SDO), D14.4 (SDI)
- new net: D14.2 (CKO), D15.5 (CKI)
- new net: D14.3 (SDO), D15.4 (SDI)
- new net CKO: D15.2 (CKO), J1.5 (Pin_5)
- new net GNDD: C1.2, C2.2, D1.6 (GND), D10.6 (GND), D11.6 (GND), D12.6 (GND), D13.6 (GND), D14.6 (GND), D15.6 (GND), D2.6 (GND), D3.6 (GND), D4.6 (GND), D5.6 (GND), D6.6 (GND), D7.6 (GND), D8.6 (GND), D9.6 (GND), J1.1 (Pin_1), J1.7 (Pin_7)
- new net POT: J2.2 (Pin_2), RV1.2
- new net SDO: D15.3 (SDO), J1.6 (Pin_6)
- new net VAA: J2.1 (Pin_1), RV1.1
Other:
- moved on the sheet: D1, D2, D3, D4
